File: hardware/trinketcore/trinketcore.kicad_sch (KiCad schematic)
At the start: 112 parts, among them J1 USB-C, J4 DISPLAY, J5 I2C OLED, J6 EXPANSION, J7 SPEAKER, J8 QWIIC, Q1 AO3401A, Q2 AO3400A, Q3 AO3400A, Q4 AO3400A, Q5 AO3401A, Q6 AO3400A, Q7 AO3401A, Q8 AO3400A, Q9 AO3400A, SW1 POWER/A, SW2 B, SW3 BOOT, SW4 RESET, U1 USBLC6-2SC6, U2 BQ25173DSGR, U3 TPS3808G01DBVR, U4 TPS63031DSKR, U5 PCF8563T, U6 RP2040, U7 W25Q128JVS, U8 MAX98357A, Y1 32.768kHz, Y2 12MHz

Commit message: TrinketCore: pin map that routes without crossings (work in progress)
The first autoroute left four connections open. Three of them were at the
RP2040, where the expansion header took GP0..GP7 in the opposite order to the
chip's pins, and USB_DET had to cross GP26/GP27 on the bottom row. The fourth
was the speaker output, hemmed in by a ground via.

- J6 now runs GP7..GP0, GP29, GP28 (pin 1 at the top), matching the pin order.
- Bottom row: CHG GP22, button A GP23, USB_DET GP24, user LED GP25 (unchanged),
  HOLD GP26, VSENSE GP27, J6 analog GP28/GP29. Display DC/CS swap to GP9/GP8.
- The amplifier's ground pins tie into its exposed pad instead of vias, and the
  RP2040 decoupling capacitors share their pins' plane vias.
- route_pcb.py runs a second Freerouting pass on the first pass's result, and
  the grid router falls back to 0.15 mm tracks.

Firmware and docs follow the new pin map. The board is being re-routed; the
board file in this commit is not routed yet.

Co-Authored-By: Claude Opus 5.5 <noreply@anthropic.com>
Claude-Session: https://claude.ai/code/session_01V89YvrQurcttiFbkgcTPH9
Connections:
- net CHG: now also U6.34 (GPIO22); no longer U6.36 (GPIO24)
- net GP0: now also J6.8 (Pin_8); no longer J6.1 (Pin_1)
- net GP1: now also J6.7 (Pin_7); no longer J6.2 (Pin_2)
- net GP2: now also J6.6 (Pin_6); no longer J6.3 (Pin_3)
- net GP3: now also J6.5 (Pin_5); no longer J6.4 (Pin_4)
- net GP4: now also J6.4 (Pin_4); no longer J6.5 (Pin_5)
- net GP5: now also J6.3 (Pin_3); no longer J6.6 (Pin_6)
- net GP6: now also J6.2 (Pin_2); no longer J6.7 (Pin_7)
- net GP7: now also J6.1 (Pin_1); no longer J6.8 (Pin_8)
- net HOLD: now also U6.38 (GPIO26_ADC0); no longer U6.34 (GPIO22)
- net TFT_CS: now also U6.11 (GPIO8); no longer U6.12 (GPIO9)
- net TFT_DC: now also U6.12 (GPIO9); no longer U6.11 (GPIO8)
- net USB_DET: now also U6.36 (GPIO24); no longer U6.40 (GPIO28_ADC2)
- net VSENSE: now also U6.39 (GPIO27_ADC1); no longer U6.41 (GPIO29_ADC3)
- net GP26 renamed GP29
- net GP29: now also U6.41 (GPIO29_ADC3); no longer U6.38 (GPIO26_ADC0)
- net GP27 renamed GP28
- net GP28: now also U6.40 (GPIO28_ADC2); no longer U6.39 (GPIO27_ADC1)
Other:
- note added: "1.8-5.5 V in, 3.3 V out, ~500 mA from a 2.6 V capacitor. VSENSE = VSYS / 2 for the RP2040's ADC (GP27)."
- note added: "J4: SPI TFT/OLED modules (GND VCC SCL SDA RES DC CS BLK). J5: I2C OLED modules (GND VCC SCL SDA). J8: Qwiic. J6: expansion (GP7-0, GP29, GP28, WAKE, VSYS, 3V3, GND)."
- note removed: "1.8-5.5 V in, 3.3 V out, ~500 mA from a 2.6 V capacitor. VSENSE = VSYS / 2 for the RP2040's ADC (GP29)."
- note removed: "J4: SPI TFT/OLED modules (GND VCC SCL SDA RES DC CS BLK). J5: I2C OLED modules (GND VCC SCL SDA). J8: Qwiic. J6: expansion (GP0-7, GP26-27, WAKE, VSYS, 3V3, GND)."
Changed lines of the file:
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@@
     )
   )
-  (text "1.8-5.5 V in, 3.3 V out, ~500 mA from a 2.6 V capacitor.\nVSENSE = VSYS / 2 for the RP2040's ADC (GP29)."
+  (text "1.8-5.5 V in, 3.3 V out, ~500 mA from a 2.6 V capacitor.\nVSENSE = VSYS / 2 for the RP2040's ADC (GP27)."
     (at 201.93 203.2 0)
     (effects
@@
     )
   )
-  (text "J4: SPI TFT/OLED modules (GND VCC SCL SDA RES DC CS BLK).\nJ5: I2C OLED modules (GND VCC SCL SDA). J8: Qwiic.\nJ6: expansion (GP0-7, GP26-27, WAKE, VSYS, 3V3, GND)."
+  (text "J4: SPI TFT/OLED modules (GND VCC SCL SDA RES DC CS BLK).\nJ5: I2C OLED modules (GND VCC SCL SDA). J8: Qwiic.\nJ6: expansion (GP7-0, GP29, GP28, WAKE, VSYS, 3V3, GND)."
     (at 400.05 287.02 0)
     (effects
@@
     (stroke (width 0) (type default))
   )
-  (label "TFT_DC"
+  (label "TFT_CS"
     (at 468.63 68.58 0)
     (fields_autoplaced)
@@
     (stroke (width 0) (type default))
   )
-  (label "TFT_CS"
+  (label "TFT_DC"
     (at 468.63 71.12 0)
     (fields_autoplaced)
@@
     (stroke (width 0) (type default))
   )
-  (label "HOLD"
+  (label "CHG"
     (at 468.63 104.14 0)
     (fields_autoplaced)
@@
     (stroke (width 0) (type default))
   )
-  (label "CHG"
+  (label "USB_DET"
     (at 468.63 109.22 0)
     (fields_autoplaced)
@@
     (stroke (width 0) (type default))
   )
-  (label "GP26"
+  (label "HOLD"
     (at 468.63 116.84 0)
     (fields_autoplaced)
@@
     (stroke (width 0) (type default))
   )
-  (label "GP27"
+  (label "VSENSE"
     (at 468.63 119.38 0)
     (fields_autoplaced)
@@
     (stroke (width 0) (type default))
   )
-  (label "USB_DET"
+  (label "GP28"
     (at 468.63 121.92 0)
     (fields_autoplaced)
@@
     (stroke (width 0) (type default))
   )
-  (label "VSENSE"
+  (label "GP29"
     (at 468.63 124.46 0)
     (fields_autoplaced)
@@
     (stroke (width 0) (type default))
   )
-  (label "GP0"
+  (label "GP7"
     (at 496.57 231.14 180)
     (fields_autoplaced)
@@
     (stroke (width 0) (type default))
   )
-  (label "GP1"
+  (label "GP6"
     (at 496.57 233.68 180)
     (fields_autoplaced)
@@
     (stroke (width 0) (type default))
   )
-  (label "GP2"
+  (label "GP5"
     (at 496.57 236.22 180)
     (fields_autoplaced)
@@
     (stroke (width 0) (type default))
   )
-  (label "GP3"
+  (label "GP4"
     (at 496.57 238.76 180)
     (fields_autoplaced)
@@
     (stroke (width 0) (type default))
   )
-  (label "GP4"
+  (label "GP3"
     (at 496.57 241.3 180)
     (fields_autoplaced)
@@
     (stroke (width 0) (type default))
   )
-  (label "GP5"
+  (label "GP2"
     (at 496.57 243.84 180)
     (fields_autoplaced)
@@
     (stroke (width 0) (type default))
   )
-  (label "GP6"
+  (label "GP1"
     (at 496.57 246.38 180)
     (fields_autoplaced)
@@
     (stroke (width 0) (type default))
   )
-  (label "GP7"
+  (label "GP0"
     (at 496.57 248.92 180)
     (fields_autoplaced)
@@
     (stroke (width 0) (type default))
   )
-  (label "GP26"
+  (label "GP29"
     (at 496.57 251.46 180)
     (fields_autoplaced)
@@
     (stroke (width 0) (type default))
   )
-  (label "GP27"
+  (label "GP28"
     (at 496.57 254 180)
     (fields_autoplaced)

Commit message: Add e-ink tarot oracle; routing fixes (work in progress)
- firmware/trinketcore/circuitpython/oracle: each press draws a random tarot
  card on a 1.54" SSD1681 e-paper module with a charge icon, then switches the
  board off (the card stays on screen with no power). make_cards.py turns card
  art into dithered 1-bit or black/white/red BMPs with the card's name.
- trinketcore.EPD_BUSY: e-paper BUSY reads on J4's BLK pin (GP13).
- READMEs and the design-method guide cover e-ink wiring and runtimes.
- route_pcb.py: the finisher now sees open connections at SMD pads (the
  report parser only matched "PTH pad"), rips up tracks around boxed-in pads
  and routes them first, and 1V1 uses the default 0.15 mm width so it fits
  between the RP2040's pins. Same parser fix in CapCore's script.
- The SWD test pads are gone (the USB bootloader is in ROM).

The board is being re-routed; the board file in this commit is not routed.

Co-Authored-By: Claude Opus 5.5 <noreply@anthropic.com>
Claude-Session: https://claude.ai/code/session_01V89YvrQurcttiFbkgcTPH9
Parts:
- removed TP1: SWCLK, TestPoint:TestPoint_Pad_D1.0mm, symbol TrinketCore:TestPoint
- removed TP2: SWDIO, TestPoint:TestPoint_Pad_D1.0mm, symbol TrinketCore:TestPoint
Other:
- note added: "12 MHz crystal, W25Q128 flash (program, sounds, pictures). BOOT + RESET: USB bootloader (SWD is not broken out). GPIO use: see the README pinout."
- note removed: "12 MHz crystal, W25Q128 flash (program, sounds, pictures). BOOT + RESET: USB bootloader. SWD on TP1/TP2. GPIO use: see the README pinout."
- moved on the sheet: C18, C19, C20, C21, C22, C23, C24, C25, C26, C27, C28, C29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
